Commit message: changed gripper

File: kinova_arm_description/description/kinova_arm.urdf (robot description, URDF)
Before this commit: robot kinova_arm, 12 links, 11 joints
Links:
- removed link gripper_base
- removed link left_gripper_finger
- removed link right_gripper_finger
- added link gripper_base_link, mass 6.6320197e-01; collision mesh filename=file:///home/chaitanya/learning/ros_workspace/install/kinov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; visual mesh filename=file:///home/chaitanya/learning/ros_workspace/install/kinov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
- added link gripper_left_finger_link, mass 4.260376752e-02; collision mesh filename=file:///home/chaitanya/learning/ros_workspace/install/kinov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; visual mesh filename=file:///home/chaitanya/learning/ros_workspace/install/kinov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
- added link gripper_left_finger_tip_link, mass 4.268588744e-02; collision mesh filename=file:///home/chaitanya/learning/ros_workspace/install/kinov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; visual mesh filename=file:///home/chaitanya/learning/ros_workspace/install/kinov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
- added link gripper_left_inner_knuckle_link, mass 2.969376448e-02; collision mesh filename=file:///home/chaitanya/learning/ros_workspace/install/kinov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; visual mesh filename=file:///home/chaitanya/learning/ros_workspace/install/kinov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
- added link gripper_left_knuckle_link, mass 1.384773208e-02; collision mesh filename=file:///home/chaitanya/learning/ros_workspace/install/kinov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; visual mesh filename=file:///home/chaitanya/learning/ros_workspace/install/kinov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
- added link gripper_right_finger_link, mass 4.260376752000000e-02; collision mesh filename=file:///home/chaitanya/learning/ros_workspace/install/kinov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; visual mesh filename=file:///home/chaitanya/learning/ros_workspace/install/kinov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
- added link gripper_right_finger_tip_link, mass 4.268588744e-02; collision mesh filename=file:///home/chaitanya/learning/ros_workspace/install/kinov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; visual mesh filename=file:///home/chaitanya/learning/ros_workspace/install/kinov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
- added link gripper_right_inner_knuckle_link, mass 2.969376448e-02; collision mesh filename=file:///home/chaitanya/learning/ros_workspace/install/kinov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; visual mesh filename=file:///home/chaitanya/learning/ros_workspace/install/kinov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
- added link gripper_right_knuckle_link, mass 1.384773208e-02; collision mesh filename=file:///home/chaitanya/learning/ros_workspace/install/kinov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; visual mesh filename=file:///home/chaitanya/learning/ros_workspace/install/kinov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
- added link kinova_camera_optical_frame
- link arm_base_link: mass None -> 50.0
Joints:
- removed joint gripper_base_joint
- removed joint left_finger_joint
- removed joint right_finger_joint
- added joint gripper_joint: type fixed, parent kinova_camera, child gripper_base_link, origin xyz=0 0.06 0 rpy=1.57 1.57 -3.14
- added joint gripper_left_finger_joint: type fixed, parent gripper_left_knuckle_link, child gripper_left_finger_link, origin xyz=0.03152616 0.0 -0.00376347 rpy=0 0 0
- added joint gripper_left_finger_tip_joint: type continuous, parent gripper_left_finger_link, child gripper_left_finger_tip_link, origin xyz=0.00563134 0.0 0.04718515 rpy=0 0 0, axis 0 -1 0, mimic joint=gripper_left_knuckle_joint multiplier=-1
- added joint gripper_left_inner_knuckle_joint: type continuous, parent gripper_base_link, child gripper_left_inner_knuckle_link, origin xyz=0.0127 0.0 0.06142 rpy=0 0 0, axis 0 -1 0, mimic joint=gripper_left_knuckle_joint
- added joint gripper_left_knuckle_joint: type revolute, parent gripper_base_link, child gripper_left_knuckle_link, origin xyz=0.03060114 0.0 0.05490452 rpy=0 0 0, axis 0 -1 0, limit lower=0.0 upper=0.8 effort=50 velocity=0.5
- added joint gripper_right_finger_joint: type fixed, parent gripper_right_knuckle_link, child gripper_right_finger_link, origin xyz=-0.03152616 0.0 -0.00376347 rpy=0 0 0
- added joint gripper_right_finger_tip_joint: type continuous, parent gripper_right_finger_link, child gripper_right_finger_tip_link, origin xyz=-0.00563134 0.0 0.04718515 rpy=0 0 0, axis 0 -1 0, mimic joint=gripper_left_knuckle_joint
- added joint gripper_right_inner_knuckle_joint: type continuous, parent gripper_base_link, child gripper_right_inner_knuckle_link, origin xyz=-0.0127 0.0 0.06142 rpy=0 0 0, axis 0 -1 0, mimic joint=gripper_left_knuckle_joint multiplier=-1
- added joint gripper_right_knuckle_joint: type revolute, parent gripper_base_link, child gripper_right_knuckle_link, origin xyz=-0.03060114 0.0 0.05490452 rpy=0 0 0, axis 0 -1 0, limit lower=-0.8 upper=0.0 effort=50 velocity=0.5, mimic joint=gripper_left_knuckle_joint multiplier=-1
- added joint kinova_camera_optical_joint: type fixed, parent kinova_camera, child kinova_camera_optical_frame, origin xyz=0 0 0 rpy=0 1.57 1.57

File: kinova_arm_description/description/kinova_arm.urdf.xacro (robot description, xacro)
@@ -10,5 +10,5 @@
     <xacro:include filename="arm/kinova_camera.xacro"/>
     <xacro:include filename="gripper/gripper_base.xacro"/>
-    <xacro:include filename="gripper/gripper_finger.xacro"/>
+    <xacro:include filename="robotiq_gripper/robotiq_gripper.xacro"/>
     <xacro:include filename="kinova_arm_gazebo.xacro"/>
     <xacro:include filename="$(find kinova_arm_moveit_config)/config/kinova_arm.ros2_control.xacro"/>
@@ -79,25 +79,9 @@
         <axis xyz="0.0 1.0 0.0"/>
     </joint>
-    <xacro:gripper_base />
-    <joint name="gripper_base_joint" type="fixed">
-        <origin xyz="0 0.062 0" rpy="0 1.57 0"/>
+    <xacro:robotiq_gripper name="gripper"/>
+    <joint name="gripper_joint" type="fixed">
+        <origin xyz="0 0.06 0" rpy="1.57 1.57 -3.14"/>
         <parent link="kinova_camera"/>
-        <child link="gripper_base"/>
-    </joint>
-    <xacro:gripper_finger name="left"/>
-    <joint name="left_finger_joint" type="prismatic">
-        <origin xyz="-0.027 0.03 0" rpy="0 1.57 1.57"/>
-        <parent link="gripper_base"/>
-        <child link="left_gripper_finger"/>
-        <axis xyz="0.0 1.0 0.0"/>
-        <limit lower="-0.026" upper="0.0" effort="1000" velocity="1000"/>
-    </joint>
-    <xacro:gripper_finger name="right"/>
-    <joint name="right_finger_joint" type="prismatic">
-        <origin xyz="0.027 0.03 0" rpy="-1.57 -1.57 0"/>
-        <parent link="gripper_base"/>
-        <child link="right_gripper_finger"/>
-        <axis xyz="0.0 1.0 0.0"/>
-        <limit lower="-0.026" upper="0.0" effort="1000" velocity="1000"/>
+        <child link="gripper_base_link"/>
     </joint>
     <link name="kinova_camera_optical_frame"/>

File: kinova_arm_moveit_config/config/kinova_arm.ros2_control.xacro (robot description, xacro)
@@ -64,17 +64,9 @@
                 <state_interface name="velocity"/>
             </joint>
-            <joint name="left_finger_joint">
+            <joint name="gripper_left_knuckle_joint">
                 <command_interface name="position"/>
                 <command_interface name="velocity"/>
                 <state_interface name="position">
-                  <param name="initial_value">${initial_positions['left_finger_joint']}</param>
-                </state_interface>
-                <state_interface name="velocity"/>
-            </joint>
-            <joint name="right_finger_joint">
-                <command_interface name="position"/>
-                <command_interface name="velocity"/>
-                <state_interface name="position">
-                  <param name="initial_value">${initial_positions['right_finger_joint']}</param>
+                  <param name="initial_value">${initial_positions['gripper_left_knuckle_joint']}</param>
                 </state_interface>
                 <state_interface name="velocity"/>
