Commit message: created kinova arm macro

File: kinova_arm_description/description/kinova_arm.urdf.xacro (robot description, xacro)
@@ -1,16 +1,11 @@
 <?xml version="1.0"?>
 <robot name="kinova_arm" xmlns:xacro="http://www.ros.org/wiki/xacro">
-    <xacro:include filename="arm/kinova_base.xacro"/>
-    <xacro:include filename="arm/kinova_shoulder.xacro"/>
-    <xacro:include filename="arm/kinova_half_arm_one.xacro"/>
-    <xacro:include filename="arm/kinova_half_arm_two.xacro"/>
-    <xacro:include filename="arm/kinova_fore_arm.xacro"/>
-    <xacro:include filename="arm/kinova_spherical_wrist_one.xacro"/>
-    <xacro:include filename="arm/kinova_spherical_wrist_two.xacro"/>
-    <xacro:include filename="arm/kinova_camera.xacro"/>
-    <xacro:include filename="robotiq_gripper/robotiq_gripper.xacro"/>
-    <xacro:include filename="$(find kinova_arm_gazebo)/gazebo/kinova_arm_gazebo.xacro"/>
-    <xacro:include filename="$(find kinova_arm_moveit_config)/config/kinova_arm.ros2_control.xacro"/>
-    <xacro:kinova_arm_ros2_control name="kinova_arm" initial_positions_file="$(find kinova_arm_moveit_config)/config/initial_positions.yaml"/>
+    <xacro:include filename="$(find kinova_arm_description)/description/kinova_arm_macro.xacro"/>
+    <xacro:kinova_arm/>
+    <joint name="arm_base_joint" type="fixed">
+            <origin xyz="0.0 0.0 0.0" rpy="1.57 0.0 3.14"/>
+            <parent link="arm_base_link"/>
+            <child link="kinova_base"/>
+    </joint>
     <link name="arm_base_link">
         <inertial>
@@ -20,73 +15,3 @@
         </inertial>
     </link>
-    <xacro:kinova_base/>
-    <joint name="arm_base_joint" type="fixed">
-        <origin xyz="0.0 0.0 0.0" rpy="1.57 0.0 3.14"/>
-        <parent link="arm_base_link"/>
-        <child link="kinova_base"/>
-    </joint>
-    <xacro:kinova_shoulder/>
-    <joint name="shoulder_joint" type="continuous">
-        <origin xyz="0 0.154 0" rpy="0 0 0"/>
-        <parent link="kinova_base"/>
-        <child link="kinova_shoulder"/>
-        <axis xyz="0.0 1.0 0.0"/>
-    </joint>
-    <xacro:kinova_half_arm_one/>
-    <joint name="half_arm_one_joint" type="revolute">
-        <origin xyz="0 0.126 0" rpy="0 0 0"/>
-        <parent link="kinova_shoulder"/>
-        <child link="kinova_half_arm_one"/>
-        <axis xyz="0.0 0.0 1.0"/>
-        <limit lower="-2.249729" upper="2.249729" effort="1000" velocity="1000"/>
-    </joint>
-    <xacro:kinova_half_arm_two/>
-    <joint name="half_arm_two_joint" type="continuous">
-        <origin xyz="0 0.2 -0.011" rpy="0 0 0"/>
-        <parent link="kinova_half_arm_one"/>
-        <child link="kinova_half_arm_two"/>
-        <axis xyz="0.0 1.0 0.0"/>
-    </joint>
-    <xacro:kinova_fore_arm/>
-    <joint name="fore_arm_joint" type="revolute">
-        <origin xyz="0 0.22 0" rpy="0 0 0"/>
-        <parent link="kinova_half_arm_two"/>
-        <child link="kinova_fore_arm"/>
-        <axis xyz="0.0 0.0 1.0"/>
-        <limit lower="-2.579597" upper="2.579597" effort="1000" velocity="1000"/>
-    </joint>
-    <xacro:kinova_spherical_wrist_one/>
-    <joint name="spherical_wrist_one_joint" type="continuous">
-        <origin xyz="0 0.21 -0.012" rpy="0 0 0"/>
-        <parent link="kinova_fore_arm"/>
-        <child link="kinova_spherical_wrist_one"/>
-        <axis xyz="0.0 1.0 0.0"/>
-    </joint>
-    <xacro:kinova_spherical_wrist_two/>
-    <joint name="spherical_wrist_two_joint" type="revolute">
-        <origin xyz="0 0.1035 0" rpy="0 0 0"/>
-        <parent link="kinova_spherical_wrist_one"/>
-        <child link="kinova_spherical_wrist_two"/>
-        <axis xyz="0.0 0.0 1.0"/>
-        <limit lower="-2.099631" upper="2.099631" effort="1000" velocity="1000"/>
-    </joint>
-    <xacro:kinova_camera/>
-    <joint name="camera_joint" type="continuous">
-        <origin xyz="0 0.11 0" rpy="0 0 0"/>
-        <parent link="kinova_spherical_wrist_two"/>
-        <child link="kinova_camera"/>
-        <axis xyz="0.0 1.0 0.0"/>
-    </joint>
-    <xacro:robotiq_gripper name="gripper"/>
-    <joint name="gripper_joint" type="fixed">
-        <origin xyz="0 0.06 0" rpy="1.57 1.57 -3.14"/>
-        <parent link="kinova_camera"/>
-        <child link="gripper_base_link"/>
-    </joint>
-    <link name="kinova_camera_optical_frame"/>
-    <joint name="kinova_camera_optical_joint" type="fixed">
-        <origin xyz="0 0 0" rpy="0 1.57 1.57"/>
-        <parent link="kinova_camera"/>
-        <child link="kinova_camera_optical_frame"/>
-    </joint>
 </robot>

Commit message: Major changes in ros control

File: kinova_arm_description/description/kinova_arm.urdf.xacro (robot description, xacro)
@@ -2,4 +2,6 @@
 <robot name="kinova_arm" xmlns:xacro="http://www.ros.org/wiki/xacro">
     <xacro:include filename="$(find kinova_arm_description)/description/kinova_arm_macro.xacro"/>
+    <xacro:include filename="$(find kinova_arm_gazebo)/gazebo/kinova_arm_ros2_control.xacro"/>
+    <xacro:kinova_arm_ros2_control name="kinova_arm" initial_positions_file="$(find kinova_arm_gazebo)/config/initial_positions.yaml"/>
     <xacro:kinova_arm/>
     <joint name="arm_base_joint" type="fixed">

File: kinova_arm_description/description/kinova_arm_macro.xacro (robot description, xacro)
@@ -12,6 +12,4 @@
         <xacro:include filename="$(find kinova_arm_description)/description/robotiq_gripper/robotiq_gripper.xacro"/>
         <xacro:include filename="$(find kinova_arm_gazebo)/gazebo/kinova_arm_gazebo.xacro"/>
-        <xacro:include filename="$(find kinova_arm_moveit_config)/config/kinova_arm.ros2_control.xacro"/>
-        <xacro:kinova_arm_ros2_control name="kinova_arm" initial_positions_file="$(find kinova_arm_moveit_config)/config/initial_positions.yaml"/>
         <xacro:kinova_base/>
         <xacro:kinova_shoulder/>

File: kinova_arm_gazebo/gazebo/kinova_arm_gazebo.xacro (robot description, xacro)
@@ -1,9 +1,4 @@
 <?xml version="1.0"?>
 <robot xmlns:xacro="http://www.ros.org/wiki/xacro" name="robot">
-    <gazebo>
-        <plugin name="gazebo_ros2_control" filename="libgazebo_ros2_control.so">
-            <parameters>$(find kinova_arm_moveit_config)/config/ros2_controllers.yaml</parameters>
-        </plugin>
-    </gazebo>
     <gazebo reference="kinova_camera">
         <sensor type="depth" name="arm_camera">

File: skratch_description/description/skratch_robot.urdf.xacro (robot description, xacro)
@@ -9,4 +9,6 @@
     <xacro:include filename="base/skratch_arm_base_plate.xacro"/>
     <xacro:include filename="$(find kinova_arm_description)/description/kinova_arm_macro.xacro"/>
+    <xacro:include filename="$(find skratch_gazebo)/gazebo/skratch_ros2_control.xacro"/>
+    <xacro:skratch_ros_control name="skratch_ros_control" initial_positions_file="$(find kinova_arm_gazebo)/config/initial_positions.yaml"/>
     <link name="base_link"></link>
     <xacro:skratch_top_base name="skratch_left_top_base"/>

File: skratch_gazebo/gazebo/skratch_gazebo.xacro (robot description, xacro)
@@ -1,5 +1,5 @@
 <?xml version="1.0"?>
 <robot xmlns:xacro="http://www.ros.org/wiki/xacro" name="robot">
-    <gazebo>
+    <!-- <gazebo>
         <plugin name="object_controller" filename="libgazebo_ros_planar_move.so">
                 <ros>
@@ -14,5 +14,5 @@
                 <publishOdomTf>true</publishOdomTf>
             </plugin>
-    </gazebo>
+    </gazebo> -->
     <gazebo reference="front_lidar">
         <sensor type="ray" name="front_lidar">

File: skratch_gazebo/gazebo/skratch_ros2_control.xacro (robot description, xacro)
@@ -1,9 +1,13 @@
 <?xml version="1.0"?>
-<robot xmlns:xacro="http://www.ros.org/wiki/xacro">
-    <xacro:macro name="kinova_arm_ros2_control" params="name initial_positions_file">
+<robot xmlns:xacro="http://www.ros.org/wiki/xacro" name="robot">
+    <gazebo>
+        <plugin name="gazebo_ros2_control" filename="libgazebo_ros2_control.so">
+            <parameters>$(find skratch_ros_control)/config/skratch_controller.yaml</parameters>
+        </plugin>
+    </gazebo>
+    <xacro:macro name="skratch_ros_control" params="name initial_positions_file">
         <xacro:property name="initial_positions" value="${load_yaml(initial_positions_file)['initial_positions']}"/>
         <ros2_control name="${name}" type="system">
             <hardware>
-                <!-- By default, set up controllers for simulation. This won't work on real hardware -->
                 <plugin>gazebo_ros2_control/GazeboSystem</plugin>
             </hardware>
@@ -72,4 +76,52 @@
                 <state_interface name="velocity"/>
             </joint>
+            <joint name="front_left_drive_left_hub_wheel_joint">
+                <command_interface name="position"/>
+                <command_interface name="velocity"/>
+                <state_interface name="position"/>
+                <state_interface name="velocity"/>
+            </joint>
+            <joint name="front_left_drive_right_hub_wheel_joint">
+                <command_interface name="position"/>
+                <command_interface name="velocity"/>
+                <state_interface name="position"/>
+                <state_interface name="velocity"/>
+            </joint>
+            <joint name="front_right_drive_left_hub_wheel_joint">
+                <command_interface name="position"/>
+                <command_interface name="velocity"/>
+                <state_interface name="position"/>
+                <state_interface name="velocity"/>
+            </joint>
+            <joint name="front_right_drive_right_hub_wheel_joint">
+                <command_interface name="position"/>
+                <command_interface name="velocity"/>
+                <state_interface name="position"/>
+                <state_interface name="velocity"/>
+            </joint>
+            <joint name="rear_left_drive_left_hub_wheel_joint">
+                <command_interface name="position"/>
+                <command_interface name="velocity"/>
+                <state_interface name="position"/>
+                <state_interface name="velocity"/>
+            </joint>
+            <joint name="rear_left_drive_right_hub_wheel_joint">
+                <command_interface name="position"/>
+                <command_interface name="velocity"/>
+                <state_interface name="position"/>
+                <state_interface name="velocity"/>
+            </joint>
+            <joint name="rear_right_drive_left_hub_wheel_joint">
+                <command_interface name="position"/>
+                <command_interface name="velocity"/>
+                <state_interface name="position"/>
+                <state_interface name="velocity"/>
+            </joint>
+            <joint name="rear_right_drive_right_hub_wheel_joint">
+                <command_interface name="position"/>
+                <command_interface name="velocity"/>
+                <state_interface name="position"/>
+                <state_interface name="velocity"/>
+            </joint>
         </ros2_control>
     </xacro:macro>
