Commit message: create ros controller for base

File: skratch_description/description/skratch_base_ros2_control.xacro (robot description, xacro)
@@ -3,7 +3,7 @@
     <ros2_control name="GazeboSystem" type="system">
         <hardware>
-            <plugin>gz_ros2_control/GazeboSimSystem</plugin>
+            <plugin>gazebo_ros2_control/GazeboSystem</plugin>
         </hardware>
-        <joint name="front_left_wheel_drive_wheel_left_joint">
+        <joint name="front_left_drive_left_hub_wheel_joint">
             <command_interface name="velocity"/>
             <command_interface name="position"/>
@@ -11,5 +11,5 @@
             <state_interface name="velocity"/>
         </joint>
-        <joint name="front_left_wheel_drive_wheel_right_joint">
+        <joint name="front_left_drive_right_hub_wheel_joint">
             <command_interface name="velocity"/>
             <command_interface name="position"/>
@@ -17,5 +17,5 @@
             <state_interface name="velocity"/>
         </joint>
-        <joint name="front_left_wheel_drive_joint">
+        <joint name="front_left_drive_pivot_joint">
             <command_interface name="velocity"/>
             <command_interface name="position"/>
@@ -23,5 +23,5 @@
             <state_interface name="velocity"/>
         </joint>
-        <joint name="front_right_wheel_drive_wheel_left_joint">
+        <joint name="front_right_drive_left_hub_wheel_joint">
             <command_interface name="velocity"/>
             <command_interface name="position"/>
@@ -29,5 +29,5 @@
             <state_interface name="velocity"/>
         </joint>
-        <joint name="front_right_wheel_drive_wheel_right_joint">
+        <joint name="front_right_drive_right_hub_wheel_joint">
             <command_interface name="velocity"/>
             <command_interface name="position"/>
@@ -35,5 +35,5 @@
             <state_interface name="velocity"/>
         </joint>
-        <joint name="front_right_wheel_drive_joint">
+        <joint name="front_right_drive_pivot_joint">
             <command_interface name="velocity"/>
             <command_interface name="position"/>
@@ -41,5 +41,5 @@
             <state_interface name="velocity"/>
         </joint>
-        <joint name="rear_left_wheel_drive_wheel_left_joint">
+        <joint name="rear_left_drive_left_hub_wheel_joint">
             <command_interface name="velocity"/>
             <command_interface name="position"/>
@@ -47,5 +47,5 @@
             <state_interface name="velocity"/>
         </joint>
-        <joint name="rear_left_wheel_drive_wheel_right_joint">
+        <joint name="rear_left_drive_right_hub_wheel_joint">
             <command_interface name="velocity"/>
             <command_interface name="position"/>
@@ -53,5 +53,5 @@
             <state_interface name="velocity"/>
         </joint>
-        <joint name="rear_left_wheel_drive_joint">
+        <joint name="rear_left_drive_pivot_joint">
             <command_interface name="velocity"/>
             <command_interface name="position"/>
@@ -59,5 +59,5 @@
             <state_interface name="velocity"/>
         </joint>
-        <joint name="rear_right_wheel_drive_wheel_left_joint">
+        <joint name="rear_right_drive_left_hub_wheel_joint">
             <command_interface name="velocity"/>
             <command_interface name="position"/>
@@ -65,5 +65,5 @@
             <state_interface name="velocity"/>
         </joint>
-        <joint name="rear_right_wheel_drive_wheel_right_joint">
+        <joint name="rear_right_drive_right_hub_wheel_joint">
             <command_interface name="velocity"/>
             <command_interface name="position"/>
@@ -71,5 +71,5 @@
             <state_interface name="velocity"/>
         </joint>
-        <joint name="rear_right_wheel_drive_joint">
+        <joint name="rear_right_drive_pivot_joint">
             <command_interface name="velocity"/>
             <command_interface name="position"/>

File: skratch_description/description/skratch_robot.urdf.xacro (robot description, xacro)
@@ -6,4 +6,5 @@
     <xacro:include filename="wheels/kelo_drive_top_part.xacro"/>
     <xacro:include filename="lidar/lidar.xacro"/>
+    <xacro:include filename="$(find skratch_description)/description/skratch_base_ros2_control.xacro"/>
     <xacro:include filename="$(find skratch_gazebo)/gazebo/skratch_gazebo.xacro"/>
     <xacro:include filename="base/skratch_arm_base_plate.xacro"/>

File: skratch_gazebo/gazebo/skratch_gazebo.xacro (robot description, xacro)
@@ -1,5 +1,5 @@
 <?xml version="1.0"?>
 <robot xmlns:xacro="http://www.ros.org/wiki/xacro" name="robot">
-    <gazebo>
+    <!-- <gazebo>
         <plugin name="object_controller" filename="libgazebo_ros_planar_move.so">
             <ros>
@@ -13,4 +13,9 @@
             <odometryRate>20.0</odometryRate>
             <publishOdomTf>true</publishOdomTf>
+        </plugin>
+    </gazebo> -->
+    <gazebo>
+        <plugin name="skratch_base_ros2_control" filename="libgazebo_ros2_control.so">
+            <parameters>$(find skratch_gazebo)/config/skratch_base_controller.yaml</parameters>
         </plugin>
     </gazebo>
