Commit message: updated the wheels xacro

File: skratch_description/description/skratch_robot.urdf.xacro (robot description, xacro)
@@ -5,7 +5,9 @@
     <xacro:include filename="base/skratch_wheel_support.xacro"/>
     <xacro:include filename="wheels/skratch_wheel_drive.xacro"/>
+    <xacro:include filename="wheels/skratch_wheel_drive_top_part.xacro"/>
     <xacro:include filename="lidar/lidar.xacro"/>
     <xacro:include filename="$(find skratch_gazebo)/gazebo/skratch_gazebo.xacro"/>
     <xacro:include filename="base/skratch_arm_base_plate.xacro"/>
+    <!-- <xacro:include filename="skratch_base_ros2_control.xacro"/> -->
     <xacro:include filename="$(find kinova_arm_description)/description/kinova_arm.urdf.xacro"/>
     <link name="base_link"></link>
@@ -58,33 +60,61 @@
         <axis xyz="0.0 0.0 1.0"/>
     </joint>
-    <xacro:skratch_wheel_drive name="front_left_wheel_drive" parent="skratch_left_wheel_support" />
+    <xacro:skratch_wheel_drive_top_part name="front_left_wheel_drive_top_part"/>
+    <joint name="front_left_wheel_drive_top_part_joint" type="fixed">
+        <origin xyz="0.202 0.0 0.018" rpy="3.14 0.0 0.0"/>
+        <parent link="skratch_left_wheel_support"/>
+        <child link="front_left_wheel_drive_top_part"/>
+        <axis xyz="0.0 0.0 1.0"/>
+    </joint>
+    <xacro:skratch_wheel_drive name="front_left_wheel_drive" parent="front_left_wheel_drive_top_part"/>
+    <!-- <joint name="front_left_wheel_drive_joint" type="continuous"> -->
     <joint name="front_left_wheel_drive_joint" type="fixed">
-    <!-- <joint name="front_left_wheel_drive_joint" type="continuous"> -->
-        <origin xyz="0.2 0.0 0.018" rpy="3.14 0.0 0.0"/>
-        <parent link="skratch_left_wheel_support"/>
+        <origin xyz="0.0 0.0 -0.09" rpy="0.0 0.0 0.0"/>
+        <parent link="front_left_wheel_drive_top_part"/>
         <child link="front_left_wheel_drive"/>
         <axis xyz="0.0 0.0 1.0"/>
     </joint>
-    <xacro:skratch_wheel_drive name="front_right_wheel_drive" parent="skratch_right_wheel_support" />
+    <xacro:skratch_wheel_drive_top_part name="front_right_wheel_drive_top_part"/>
+    <joint name="front_right_wheel_drive_top_part_joint" type="fixed">
+        <origin xyz="-0.202 0.0 0.018" rpy="3.14 0.0 0.0"/>
+        <parent link="skratch_right_wheel_support"/>
+        <child link="front_right_wheel_drive_top_part"/>
+        <axis xyz="0.0 0.0 1.0"/>
+    </joint>
+    <xacro:skratch_wheel_drive name="front_right_wheel_drive" parent="front_right_wheel_drive_top_part"/>
+    <!-- <joint name="front_right_wheel_drive_joint" type="continuous"> -->
     <joint name="front_right_wheel_drive_joint" type="fixed">
-    <!-- <joint name="front_right_wheel_drive_joint" type="continuous"> -->
-        <origin xyz="-0.2 0.0 0.018" rpy="3.14 0.0 0.0"/>
-        <parent link="skratch_right_wheel_support"/>
+        <origin xyz="0.0 0.0 -0.09" rpy="0.0 0.0 0.0"/>
+        <parent link="front_right_wheel_drive_top_part"/>
         <child link="front_right_wheel_drive"/>
         <axis xyz="0.0 0.0 1.0"/>
     </joint>
-    <xacro:skratch_wheel_drive name="rear_left_wheel_drive" parent="skratch_left_wheel_support"/>
+    <xacro:skratch_wheel_drive_top_part name="rear_left_wheel_drive_top_part"/>
+    <joint name="rear_left_wheel_drive_top_part_joint" type="fixed">
+        <origin xyz="-0.202 0.0 0.018" rpy="3.14 0.0 0.0"/>
+        <parent link="skratch_left_wheel_support"/>
+        <child link="rear_left_wheel_drive_top_part"/>
+        <axis xyz="0.0 0.0 1.0"/>
+    </joint>
+    <xacro:skratch_wheel_drive name="rear_left_wheel_drive" parent="rear_left_wheel_drive_top_part"/>
+    <!-- <joint name="rear_left_wheel_drive_joint" type="continuous"> -->
     <joint name="rear_left_wheel_drive_joint" type="fixed">
-    <!-- <joint name="rear_left_wheel_drive_joint" type="continuous"> -->
-        <origin xyz="-0.2 0.0 0.018" rpy="3.14 0.0 0.0"/>
-        <parent link="skratch_left_wheel_support"/>
+        <origin xyz="0.0 0.0 -0.09" rpy="0.0 0.0 0.0"/>
+        <parent link="rear_left_wheel_drive_top_part"/>
         <child link="rear_left_wheel_drive"/>
         <axis xyz="0.0 0.0 1.0"/>
     </joint>
-    <xacro:skratch_wheel_drive name="rear_right_wheel_drive" parent="skratch_right_wheel_support"/>
+    <xacro:skratch_wheel_drive_top_part name="rear_right_wheel_drive_top_part"/>
+    <joint name="rear_right_wheel_drive_top_part_joint" type="fixed">
+        <origin xyz="0.202 0.0 0.018" rpy="3.14 0.0 0.0"/>
+        <parent link="skratch_right_wheel_support"/>
+        <child link="rear_right_wheel_drive_top_part"/>
+        <axis xyz="0.0 0.0 1.0"/>
+    </joint>
+    <xacro:skratch_wheel_drive name="rear_right_wheel_drive" parent="rear_right_wheel_drive_top_part"/>
+    <!-- <joint name="rear_right_wheel_drive_joint" type="continuous"> -->
     <joint name="rear_right_wheel_drive_joint" type="fixed">
-    <!-- <joint name="rear_right_wheel_drive_joint" type="continuous"> -->
-        <origin xyz="0.2 0.0 0.018" rpy="3.14 0.0 0.0"/>
-        <parent link="skratch_right_wheel_support"/>
+        <origin xyz="0.0 0.0 -0.09" rpy="0.0 0.0 0.0"/>
+        <parent link="rear_right_wheel_drive_top_part"/>
         <child link="rear_right_wheel_drive"/>
         <axis xyz="0.0 0.0 1.0"/>

File: skratch_description/description/wheels/skratch_wheel.xacro (robot description, xacro)
@@ -2,21 +2,9 @@
 <robot name="skratch_wheel" xmlns:xacro="http://www.ros.org/wiki/xacro">
     <xacro:macro name="skratch_wheel" params="name parent">
-        <!-- <xacro:if value="${movable_joints}">
-            <transmission name="${name}_transmission">
-                <type>transmission_interface/SimpleTransmission</type>
-                <joint name="${name}_joint">
-                    <hardwareInterface>hardware_interface/EffortJointInterface</hardwareInterface>
-                </joint>
-                <actuator name="${name}_motor">
-                    <mechanicalReduction>1.0</mechanicalReduction>
-                    <hardwareInterface>hardware_interface/EffortJointInterface</hardwareInterface>
-                </actuator>
-            </transmission>
-        </xacro:if> -->
         <link name="${name}">
             <inertial>
-                <origin xyz="0.0 0.0 0.0" rpy="0.0 -0.0 0.0" />
-                <mass value="0.25" />
-                <inertia ixx="0.0001913" iyy="0.0001913" izz="0.0003315" ixy="0.0" iyz="0.0" ixz="0.0" />
+                <origin xyz="0 0 0" rpy="0 0 0"/>
+                <mass value="1.56317"/>
+                <inertia ixx="0.00101253363" ixy="0.00000000000" ixz="0.00000001020" iyy="0.00157998524" iyz="-0.00000055474" izz="0.00101282739"/>
             </inertial>
             <visual>

File: skratch_description/description/wheels/skratch_wheel_drive.xacro (robot description, xacro)
@@ -3,26 +3,14 @@
     <xacro:macro name="skratch_wheel_drive" params="name parent">
         <xacro:include filename="wheels/skratch_wheel.xacro"/>
-        <!-- <xacro:if value="${movable_joints}">
-            <transmission name="${name}_transmission">
-                <type>transmission_interface/SimpleTransmission</type>
-                <joint name="${name}_pivot_joint">
-                    <hardwareInterface>hardware_interface/EffortJointInterface</hardwareInterface>
-                </joint>
-                <actuator name="${name}_pivot_motor">
-                    <mechanicalReduction>1.0</mechanicalReduction>
-                    <hardwareInterface>hardware_interface/EffortJointInterface</hardwareInterface>
-                </actuator>
-            </transmission>
-        </xacro:if> -->
         <link name="${name}">
             <inertial>
-                <origin xyz="0.0 0.0 0.0" rpy="0.0 0.0 1.57" />
-                <mass value="0.5" />
-                <inertia ixx="0.001773" iyy="0.001755" izz="0.001341" ixy="0.0" iyz="0.0" ixz="0.0" />
+                <origin xyz="0.00023 -0.00095 0.04843" rpy="0 0 0"/>
+                <mass value="1.46273"/>
+                <inertia ixx="0.00302046423" ixy="0.00000851844" ixz="0.00001188180" iyy="0.00326495472" iyz="0.00001855408" izz="0.00386072964"/>
             </inertial>
             <visual>
-                <origin xyz="0.0 0.0 0.0" rpy="0.0 0.0 1.57" />
+                <origin xyz="0.0 0.0 0.0" rpy="0.0 0.0 0.0" />
                 <geometry>
-                    <mesh filename="file://$(find skratch_description)/meshes/wheels/kelo_drive_base.stl" scale="0.001 0.001 0.001"/>
+                    <mesh filename="file://$(find skratch_description)/meshes/wheels/kelo_drive_mid_part.dae" scale="1 1 1"/>
                 </geometry>
                 <material name="LightGrey">
@@ -33,5 +21,5 @@
                 <origin xyz="0.0 0.0 0.0" rpy="0.0 0.0 0.0" />
                 <geometry>
-                    <mesh filename="file://$(find skratch_description)/meshes/wheels/kelo_drive_base.stl" scale="0.001 0.001 0.001"/>
+                    <mesh filename="file://$(find skratch_description)/meshes/wheels/kelo_drive_mid_part.dae" scale="1 1 1"/>
                 </geometry>
             </collision>
@@ -42,10 +30,9 @@
         <xacro:skratch_wheel name="${name}_wheel_left" parent="${name}"/>
         <joint name="${name}_wheel_left_joint" type="continuous">
-        <!-- <joint name="${name}_wheel_left_joint" type="fixed"> -->
-            <origin xyz="0.01 0.04 -0.09" rpy="0.0 0.0 0.0"/>
+            <origin xyz="0.0 0.04 0.0" rpy="0.0 0.0 0.0"/>
             <parent link="${name}"/>
             <child link="${name}_wheel_left"/>
             <axis xyz="0.0 1.0 0.0"/>
-            <gazebo>
+            <!-- <gazebo>
                 <mu1>1.0</mu1>
                 <mu2>1.0</mu2>
@@ -53,14 +40,13 @@
                 <kd>1.0</kd>
                 <fdir1>0 0 0</fdir1>
-            </gazebo>
+            </gazebo> -->
         </joint>
         <xacro:skratch_wheel name="${name}_wheel_right" parent="${name}"/>
         <joint name="${name}_wheel_right_joint" type="continuous">
-        <!-- <joint name="${name}_wheel_right_joint" type="fixed"> -->
-            <origin xyz="0.01 -0.04 -0.09" rpy="0.0 0.0 0.0"/>
+            <origin xyz="0.0 -0.04 0.0" rpy="0.0 0.0 0.0"/>
             <parent link="${name}"/>
             <child link="${name}_wheel_right"/>
             <axis xyz="0.0 1.0 0.0"/>
-            <gazebo>
+            <!-- <gazebo>
                 <mu1>1.0</mu1>
                 <mu2>1.0</mu2>
@@ -68,5 +54,5 @@
                 <kd>1.0</kd>
                 <fdir1>0 0 0</fdir1>
-            </gazebo>
+            </gazebo> -->
         </joint>
     </xacro:macro>

Commit message: updated urdf with new macros

File: skratch_description/description/skratch_robot.urdf.xacro (robot description, xacro)
@@ -4,11 +4,9 @@
     <xacro:include filename="base/skratch_top_base.xacro"/>
     <xacro:include filename="base/skratch_wheel_support.xacro"/>
-    <xacro:include filename="wheels/skratch_wheel_drive.xacro"/>
-    <xacro:include filename="wheels/skratch_wheel_drive_top_part.xacro"/>
+    <xacro:include filename="wheels/kelo_drive_top_part.xacro"/>
     <xacro:include filename="lidar/lidar.xacro"/>
     <xacro:include filename="$(find skratch_gazebo)/gazebo/skratch_gazebo.xacro"/>
     <xacro:include filename="base/skratch_arm_base_plate.xacro"/>
-    <!-- <xacro:include filename="skratch_base_ros2_control.xacro"/> -->
-    <xacro:include filename="$(find kinova_arm_description)/description/kinova_arm.urdf.xacro"/>
+    <xacro:include filename="$(find kinova_arm_description)/description/kinova_arm_macro.xacro"/>
     <link name="base_link"></link>
     <xacro:skratch_top_base name="skratch_left_top_base"/>
@@ -54,70 +52,22 @@
         <child link="skratch_arm_base_plate"/>
     </joint>
+    <xacro:kinova_arm/>
     <joint name="kinova_arm_base_joint" type="fixed">
-        <origin xyz="0.0 0.0 0.0" rpy="0.0 0.0 0.0"/>
+        <origin xyz="0.0 0.0 0.0" rpy="1.57 0 3.14"/>
         <parent link="skratch_arm_base_plate"/>
-        <child link="arm_base_link"/>
-        <axis xyz="0.0 0.0 1.0"/>
+        <child link="kinova_base"/>
     </joint>
-    <xacro:skratch_wheel_drive_top_part name="front_left_wheel_drive_top_part"/>
-    <joint name="front_left_wheel_drive_top_part_joint" type="fixed">
-        <origin xyz="0.202 0.0 0.018" rpy="3.14 0.0 0.0"/>
-        <parent link="skratch_left_wheel_support"/>
-        <child link="front_left_wheel_drive_top_part"/>
-        <axis xyz="0.0 0.0 1.0"/>
-    </joint>
-    <xacro:skratch_wheel_drive name="front_left_wheel_drive" parent="front_left_wheel_drive_top_part"/>
-    <!-- <joint name="front_left_wheel_drive_joint" type="continuous"> -->
-    <joint name="front_left_wheel_drive_joint" type="fixed">
-        <origin xyz="0.0 0.0 -0.09" rpy="0.0 0.0 0.0"/>
-        <parent link="front_left_wheel_drive_top_part"/>
-        <child link="front_left_wheel_drive"/>
-        <axis xyz="0.0 0.0 1.0"/>
-    </joint>
-    <xacro:skratch_wheel_drive_top_part name="front_right_wheel_drive_top_part"/>
-    <joint name="front_right_wheel_drive_top_part_joint" type="fixed">
-        <origin xyz="-0.202 0.0 0.018" rpy="3.14 0.0 0.0"/>
-        <parent link="skratch_right_wheel_support"/>
-        <child link="front_right_wheel_drive_top_part"/>
-        <axis xyz="0.0 0.0 1.0"/>
-    </joint>
-    <xacro:skratch_wheel_drive name="front_right_wheel_drive" parent="front_right_wheel_drive_top_part"/>
-    <!-- <joint name="front_right_wheel_drive_joint" type="continuous"> -->
-    <joint name="front_right_wheel_drive_joint" type="fixed">
-        <origin xyz="0.0 0.0 -0.09" rpy="0.0 0.0 0.0"/>
-        <parent link="front_right_wheel_drive_top_part"/>
-        <child link="front_right_wheel_drive"/>
-        <axis xyz="0.0 0.0 1.0"/>
-    </joint>
-    <xacro:skratch_wheel_drive_top_part name="rear_left_wheel_drive_top_part"/>
-    <joint name="rear_left_wheel_drive_top_part_joint" type="fixed">
-        <origin xyz="-0.202 0.0 0.018" rpy="3.14 0.0 0.0"/>
-        <parent link="skratch_left_wheel_support"/>
-        <child link="rear_left_wheel_drive_top_part"/>
-        <axis xyz="0.0 0.0 1.0"/>
-    </joint>
-    <xacro:skratch_wheel_drive name="rear_left_wheel_drive" parent="rear_left_wheel_drive_top_part"/>
-    <!-- <joint name="rear_left_wheel_drive_joint" type="continuous"> -->
-    <joint name="rear_left_wheel_drive_joint" type="fixed">
-        <origin xyz="0.0 0.0 -0.09" rpy="0.0 0.0 0.0"/>
-        <parent link="rear_left_wheel_drive_top_part"/>
-        <child link="rear_left_wheel_drive"/>
-        <axis xyz="0.0 0.0 1.0"/>
-    </joint>
-    <xacro:skratch_wheel_drive_top_part name="rear_right_wheel_drive_top_part"/>
-    <joint name="rear_right_wheel_drive_top_part_joint" type="fixed">
-        <origin xyz="0.202 0.0 0.018" rpy="3.14 0.0 0.0"/>
-        <parent link="skratch_right_wheel_support"/>
-        <child link="rear_right_wheel_drive_top_part"/>
-        <axis xyz="0.0 0.0 1.0"/>
-    </joint>
-    <xacro:skratch_wheel_drive name="rear_right_wheel_drive" parent="rear_right_wheel_drive_top_part"/>
-    <!-- <joint name="rear_right_wheel_drive_joint" type="continuous"> -->
-    <joint name="rear_right_wheel_drive_joint" type="fixed">
-        <origin xyz="0.0 0.0 -0.09" rpy="0.0 0.0 0.0"/>
-        <parent link="rear_right_wheel_drive_top_part"/>
-        <child link="rear_right_wheel_drive"/>
-        <axis xyz="0.0 0.0 1.0"/>
-    </joint>
+    <xacro:kelo_drive_top_part name="front_left_drive_top_part" parent="skratch_left_wheel_support" drive_name="front_left_drive">
+        <origin xyz="0.202 0 0.018" rpy="3.14 0 0.0"/>
+    </xacro:kelo_drive_top_part>
+    <xacro:kelo_drive_top_part name="front_right_drive_top_part" parent="skratch_right_wheel_support" drive_name="front_right_drive">
+        <origin xyz="-0.202 0 0.018" rpy="3.14 0 0.0"/>
+    </xacro:kelo_drive_top_part>
+    <xacro:kelo_drive_top_part name="rear_left_drive_top_part" parent="skratch_left_wheel_support" drive_name="rear_left_drive">
+        <origin xyz="-0.202 0 0.018" rpy="3.14 0 0.0"/>
+    </xacro:kelo_drive_top_part>
+    <xacro:kelo_drive_top_part name="rear_right_drive_top_part" parent="skratch_right_wheel_support" drive_name="rear_right_drive">
+        <origin xyz="0.202 0 0.018" rpy="3.14 0 0.0"/>
+    </xacro:kelo_drive_top_part>
     <xacro:lidar name="front_lidar"/>
     <joint name="front_lidar_joint" type="fixed">

Commit message: Reverted back to original control

File: skratch_description/description/skratch_robot.urdf.xacro (robot description, xacro)
@@ -9,6 +9,6 @@
     <xacro:include filename="base/skratch_arm_base_plate.xacro"/>
     <xacro:include filename="$(find kinova_arm_description)/description/kinova_arm_macro.xacro"/>
-    <xacro:include filename="$(find skratch_gazebo)/gazebo/skratch_ros2_control.xacro"/>
-    <xacro:skratch_ros_control name="skratch_ros_control" initial_positions_file="$(find kinova_arm_gazebo)/config/initial_positions.yaml"/>
+    <xacro:include filename="$(find kinova_arm_gazebo)/gazebo/kinova_arm_ros2_control.xacro"/>
+    <xacro:kinova_arm_ros2_control name="kinova_arm" initial_positions_file="$(find kinova_arm_gazebo)/config/initial_positions.yaml"/>
     <link name="base_link"></link>
     <xacro:skratch_top_base name="skratch_left_top_base"/>
@@ -60,14 +60,14 @@
         <child link="kinova_base"/>
     </joint>
-    <xacro:kelo_drive_top_part name="front_left_drive_top_part" parent="skratch_left_wheel_support" drive_name="front_left_drive">
+    <xacro:kelo_drive_top_part name="front_left_drive_top_part" parent="skratch_left_wheel_support" drive_name="skratch_1_drive">
         <origin xyz="0.202 0 0.018" rpy="3.14 0 0.0"/>
     </xacro:kelo_drive_top_part>
-    <xacro:kelo_drive_top_part name="front_right_drive_top_part" parent="skratch_right_wheel_support" drive_name="front_right_drive">
+    <xacro:kelo_drive_top_part name="front_right_drive_top_part" parent="skratch_right_wheel_support" drive_name="skratch_2_drive">
         <origin xyz="-0.202 0 0.018" rpy="3.14 0 0.0"/>
     </xacro:kelo_drive_top_part>
-    <xacro:kelo_drive_top_part name="rear_left_drive_top_part" parent="skratch_left_wheel_support" drive_name="rear_left_drive">
+    <xacro:kelo_drive_top_part name="rear_left_drive_top_part" parent="skratch_left_wheel_support" drive_name="skratch_3_drive">
         <origin xyz="-0.202 0 0.018" rpy="3.14 0 0.0"/>
     </xacro:kelo_drive_top_part>
-    <xacro:kelo_drive_top_part name="rear_right_drive_top_part" parent="skratch_right_wheel_support" drive_name="rear_right_drive">
+    <xacro:kelo_drive_top_part name="rear_right_drive_top_part" parent="skratch_right_wheel_support" drive_name="skratch_4_drive">
         <origin xyz="0.202 0 0.018" rpy="3.14 0 0.0"/>
     </xacro:kelo_drive_top_part>

File: skratch_description/description/wheels/kelo_drive.xacro (robot description, xacro)
@@ -25,10 +25,9 @@
             </inertial>
         </link>
-        <joint name="${name}_pivot_joint" type="continuous">
+        <joint name="${name}_pivot_joint" type="fixed">
             <xacro:insert_block name="origin" />
             <axis xyz="0 0 1"/>
             <parent link="${parent}"/>
             <child link="${name}_pivot_link" />
-            <dynamics damping="0.1" friction="0.05"/>
             <limit effort="2.0" velocity="1.0"/>
         </joint>

File: skratch_gazebo/gazebo/skratch_gazebo.xacro (robot description, xacro)
@@ -1,4 +1,18 @@
 <?xml version="1.0"?>
 <robot xmlns:xacro="http://www.ros.org/wiki/xacro" name="robot">
+    <gazebo>
+        <plugin name="object_controller" filename="libgazebo_ros_planar_move.so">
+            <ros>
+                <remapping>cmd_vel:=cmd_vel</remapping>
+                <remapping>odom:=odom</remapping>
+            </ros>
+            <commandTopic>cmd_vel</commandTopic>
+            <odometryTopic>odom</odometryTopic>
+            <odometryFrame>odom</odometryFrame>
+            <robotBaseFrame>base_link</robotBaseFrame>
+            <odometryRate>20.0</odometryRate>
+            <publishOdomTf>true</publishOdomTf>
+        </plugin>
+    </gazebo>
     <gazebo reference="front_lidar">
         <sensor type="ray" name="front_lidar">

Commit message: Added Battery to robot

File: skratch_description/description/skratch_robot.urdf.xacro (robot description, xacro)
@@ -7,5 +7,5 @@
     <xacro:include filename="lidar/lidar.xacro"/>
     <xacro:include filename="$(find skratch_gazebo)/gazebo/skratch_gazebo.xacro"/>
-    <xacro:include filename="base/skratch_arm_base_plate.xacro"/>
+    <xacro:include filename="base/skratch_base_plate.xacro"/>
     <xacro:include filename="$(find kinova_arm_description)/description/kinova_arm_macro.xacro"/>
     <xacro:include filename="$(find kinova_arm_gazebo)/gazebo/kinova_arm_ros2_control.xacro"/>
@@ -48,7 +48,7 @@
         <child link="skratch_right_wheel_support"/>
     </joint>
-    <xacro:skratch_arm_base_plate name="skratch_arm_base_plate"/>
+    <xacro:skratch_base_plate name="skratch_arm_base_plate"/>
     <joint name="arm_base_plate_joint" type="fixed">
-        <origin xyz="0.2115 0.0 0.023" rpy="0.0 0.0 0.0"/>
+        <origin xyz="0.2115 0.005 0.023" rpy="0.0 0.0 0.0"/>
         <parent link="skratch_left_top_base"/>
         <child link="skratch_arm_base_plate"/>
@@ -86,3 +86,38 @@
         <axis xyz="0.0 0.0 1.0"/>
     </joint>
+    <xacro:skratch_base_plate name="skratch_battery_base_plate"/>
+    <joint name="battery_base_plate_joint" type="fixed">
+        <origin xyz="-0.2115 0.005 0.023" rpy="0.0 0.0 3.1416"/>
+        <parent link="skratch_left_top_base"/>
+        <child link="skratch_battery_base_plate"/>
+    </joint>
+    <link name="battery_link">
+        <visual>
+            <geometry>
+                <box size="0.166 0.196 0.175"/>
+            </geometry>
+            <material name="battery_color">
+                <color rgba="0.0 0.0 0.0 1.0"/>
+            </material>
+        </visual>
+        <collision>
+            <geometry>
+                <box size="0.166 0.196 0.175"/>
+            </geometry>
+        </collision>
+        <inertial>
+            <origin xyz="0 0 0" rpy="0 0 0"/>
+            <mass value="7.0"/>
+            <inertia ixx="0.403" ixy="0.0" ixz="0.0" iyy="0.345" iyz="0.0" izz="0.388"/>
+        </inertial>
+    </link>
+    <gazebo reference="battery_link">
+        <material>Gazebo/Black</material>
+    </gazebo>
+    <joint name="battery_joint" type="fixed">
+        <origin xyz="0.0 0.0 0.0875" rpy="0.0 0.0 0.0"/>
+        <parent link="skratch_battery_base_plate"/>
+        <child link="battery_link"/>
+        <axis xyz="0.0 0.0 1.0"/>
+    </joint>
 </robot>
