Commit message: Renamed file

File: skratch_description/description/base/skratch_base_plate.xacro (robot description, xacro)
@@ -1,5 +1,5 @@
 <?xml version="1.0"?>
-<robot name="skratch_arm_base_plate" xmlns:xacro="http://www.ros.org/wiki/xacro">
-    <xacro:macro name="skratch_arm_base_plate" params="name">
+<robot name="skratch_arm_plate" xmlns:xacro="http://www.ros.org/wiki/xacro">
+    <xacro:macro name="skratch_base_plate" params="name">
         <link name="${name}">
             <inertial>
@@ -11,5 +11,5 @@
                 <origin xyz="0.0 0.0 0.0" rpy="0.0 0.0 1.57" />
                 <geometry>
-                    <mesh filename="file://$(find skratch_description)/meshes/base/skratch_arm_base_plate.stl" scale="0.001 0.001 0.001"/>
+                    <mesh filename="file://$(find skratch_description)/meshes/base/skratch_base_plate.stl" scale="0.001 0.001 0.001"/>
                 </geometry>
                 <material name="Grey">
@@ -20,5 +20,5 @@
                 <origin xyz="0.0 0.0 0.0" rpy="0.0 0.0 1.57" />
                 <geometry>
-                    <mesh filename="file://$(find skratch_description)/meshes/base/skratch_arm_base_plate.stl" scale="0.001 0.001 0.001"/>
+                    <mesh filename="file://$(find skratch_description)/meshes/base/skratch_base_plate.stl" scale="0.001 0.001 0.001"/>
                 </geometry>
             </collision>
