Commit message: Added color to wheels

File: skratch_description/description/wheels/kelo_drive_wheel.xacro (robot description, xacro)
@@ -24,4 +24,7 @@
             </inertial>
         </link>
+        <gazebo reference="${name}_link">
+            <material>Gazebo/Black</material>
+        </gazebo>
         <joint name="${name}_joint" type="continuous">
             <xacro:insert_block name="origin" />
